File: ANTS-Power-board.kicad_pcb (KiCad board)
At the start: 2 copper layers, 80 x 80 mm, 28 parts, among them U1 TPS62916RPYR, U2 LP2985-3.3

Commit message: Ferrite bead labeling on PCB fixed
Connections:
- C10 pad 1: 5V_out -> /5V SMPS/VO
- C11 pad 1: 5V_out -> /5V SMPS/VO
- C12 pad 1: 5V_out -> /5V SMPS/VO
- C13 pad 1: 5V_out -> /5V SMPS/VO
- C14 pad 1: 5V_out -> /5V SMPS/VO
- C7 pad 1: 5V_out -> /5V SMPS/VO
- C8 pad 1: 5V_out -> /5V SMPS/VO
- C9 pad 1: 5V_out -> /5V SMPS/VO
- FB1 pad 2: 5V_out -> /5V SMPS/VO
- L1 pad 1: 5V_out -> /5V SMPS/VO
- R2 pad 1: 5V_out -> /5V SMPS/VO
- U1 pad 4: 5V_out -> /5V SMPS/VO
Routing:
- net 5V_out: track 192.7 -> 99.4 mm
- net /5V SMPS/VO: track 0.00 -> 93.4 mm
